Commit message: added texture

File: assets/urdf/ycb/bottle/model.urdf (robot description, URDF)
Before this commit: robot mustard_bottle, 1 links, 0 joints
Links:
- link mustard_bottle__link: geometry collision mesh filename=ycb/bottle/textured.dae scale=1.0 1.0 1.0; visual mesh filename=ycb/bottle/textured.dae scale=1.0 1.0 1.0
